File: leds.kicad_sch (KiCad schematic)
At the start: 18 parts

Commit message: Prepare HPA300 hardware repository for Rev A release.
Other:
- company: (none) -> PJM
- title: (none) -> HPA300 Replacement Controller
Changed lines of the file:
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@@
 	(generator_version "9.0")
 	(paper "A4")
+	(title_block
+		(title "HPA300 Replacement Controller")
+		(date "11/12/2025")
+		(rev "A")
+		(company "PJM")
+		(comment 1 "Open hardware — CERN-OHL-W-2.0")
+		(comment 2 "github.com/patmont/HPA300-hardware")
+		(comment 3 "Independent project; not affiliated with Honeywell")
+	)
 	(text_box "LED1: FAN 3\nLED2: CHECK FILTERS\nLED3: 8h TIMER\nLED4: FAN 2\nLED5: CHECK PRE-FILTER\nLED6: 4h TIMER\nLED7: FAN 1\nLED8: FAN 4\nLED9: 2h TIMER"
 		(exclude_from_sim no)
