File: mcu.kicad_sch (KiCad schematic)
At the start: 10 parts, among them SW1 RESET, SW2 BOOT, U1 ESP32-S2-SOLO-2

Commit message: Prepare HPA300 hardware repository for Rev A release.
Other:
- company: (none) -> PJM
- title: (none) -> HPA300 Replacement Controller
Changed lines of the file:
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@@
 	(generator_version "9.0")
 	(paper "A4")
+	(title_block
+		(title "HPA300 Replacement Controller")
+		(date "11/12/2025")
+		(rev "A")
+		(company "PJM")
+		(comment 1 "Open hardware — CERN-OHL-W-2.0")
+		(comment 2 "github.com/patmont/HPA300-hardware")
+		(comment 3 "Independent project; not affiliated with Honeywell")
+	)
 	(junction
 		(at 49.53 106.68)
