File: touchkeys.kicad_sch (KiCad schematic)
At the start: 12 parts

Commit message: Prepare HPA300 hardware repository for Rev A release.
Other:
- company: (none) -> PJM
- title: (none) -> HPA300 Replacement Controller
Changed lines of the file:
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@@
 	(generator_version "9.0")
 	(paper "A4")
+	(title_block
+		(title "HPA300 Replacement Controller")
+		(date "11/12/2025")
+		(rev "A")
+		(company "PJM")
+		(comment 1 "Open hardware — CERN-OHL-W-2.0")
+		(comment 2 "github.com/patmont/HPA300-hardware")
+		(comment 3 "Independent project; not affiliated with Honeywell")
+	)
 	(text_box "Spark gap and 10k resistor for ESD protection. Place spark gap close to the touch key, place resistor close to the MCU."
 		(exclude_from_sim no)
